File: Hardware/LEDTimer/LEDTimer.kicad_pcb (KiCad board)
At the start: 4 copper layers, 38 x 27.3 mm, 37 parts, among them J2 LED, J3 PWR, Q1 S8050, SW1 SW_Push, SW2 SW_Push, SW3 SW_Push, SW4 SW_PWR, U1 AP7383-36WW7, U2 PIC16F1825, U3 Display_128x64_096_I2C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

Commit message: PCB: add interactive BOM
Parts:
- JP1: value OLED1 -> OLED_PIN1
- JP2: value OLED2 -> OLED_PIN2

Commit message: PCB: add pull-down resistor to LED_EN_PWM
Parts:
- added R5: 10k, Resistor_SMD:R_0805_2012Metric_Pad1.20x1.40mm_HandSolder, F.Cu at (141.5, 99.6)
Routing:
- net /LED_EN_PWM: track 5.36 -> 5.94 mm
- net GND: vias 14 -> 19
Changed lines of the file:
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@@
     (property "Sheetname" "")
     (attr smd)
-    (fp_text reference "C2" (at 0 -1.7 -90) (layer "F.SilkS")
+    (fp_text reference "C2" (at 2.4 0) (layer "F.SilkS")
       (effects (font (size 1 1) (thickness 0.15)))
     )
@@
     (pad "4" thru_hole oval (at 3.81 0 90) (size 1.7 1.7) (drill 1) (layers *.Cu *.Mask)
       (net 18 "Net-(R6-Pad2)") (pinfunction "SDA") (pintype "bidirectional"))
-    (model "${KIPRJMOD}/SSD1306_OLED_Display(128x64).step" hide
+    (model "${KIPRJMOD}/SSD1306_OLED_Display(128x64).step"
       (offset (xyz 0 -12 4.5))
       (scale (xyz 1 1 1))
@@
     )
   )
+  (footprint "Resistor_SMD:R_0805_2012Metric_Pad1.20x1.40mm_HandSolder" (layer "F.Cu")
+    (at 141.5 99.6 -90)
+    (descr "Resistor SMD 0805 (2012 Metric), square (rectangular) end terminal, IPC_7351 nominal with elongated pad for handsoldering. (Body size source: IPC-SM-782 page 72, https://www.pcb-3d.com/wordpress/wp-content/uploads/ipc-sm-782a_amendment_1_and_2.pdf), generated with kicad-footprint-generator")
+    (tags "resistor handsolder")
+    (property "Sheetfile" "LEDTimer.kicad_sch")
+    (property "Sheetname" "")
+    (attr smd)
+    (fp_text reference "R5" (at -2.3 0 180) (layer "F.SilkS")
+      (effects (font (size 1 1) (thickness 0.15)))
+    )
+    (fp_text value "10k" (at 0 1.65 90) (layer "F.Fab")
+      (effects (font (size 1 1) (thickness 0.15)))
+    )
+    (fp_text user "${REFERENCE}" (at 0 0 90) (layer "F.Fab")
+      (effects (font (size 0.5 0.5) (thickness 0.08)))
+    )
+    (fp_line (start -0.227064 -0.735) (end 0.227064 -0.735) (layer "F.SilkS") (width 0.12))
+    (fp_line (start -0.227064 0.735) (end 0.227064 0.735) (layer "F.SilkS") (width 0.12))
+    (fp_line (start -1.85 -0.95) (end 1.85 -0.95) (layer "F.CrtYd") (width 0.05))
+    (fp_line (start -1.85 0.95) (end -1.85 -0.95) (layer "F.CrtYd") (width 0.05))
+    (fp_line (start 1.85 0.95) (end -1.85 0.95) (layer "F.CrtYd") (width 0.05))
+    (fp_line (start 1.85 -0.95) (end 1.85 0.95) (layer "F.CrtYd") (width 0.05))
+    (fp_line (start 1 -0.625) (end 1 0.625) (layer "F.Fab") (width 0.1))
+    (fp_line (start -1 0.625) (end -1 -0.625) (layer "F.Fab") (width 0.1))
+    (fp_line (start 1 0.625) (end -1 0.625) (layer "F.Fab") (width 0.1))
+    (fp_line (start -1 -0.625) (end 1 -0.625) (layer "F.Fab") (width 0.1))
+    (pad "1" smd roundrect (at -1 0 270) (size 1.2 1.4) (layers "F.Cu" "F.Paste" "F.Mask") (roundrect_rratio 0.208333)
+      (net 13 "/LED_EN_PWM") (pintype "passive"))
+    (pad "2" smd roundrect (at 1 0 270) (size 1.2 1.4) (layers "F.Cu" "F.Paste" "F.Mask") (roundrect_rratio 0.208333)
+      (net 2 "GND") (pintype "passive"))
+    (model "${KICAD6_3DMODEL_DIR}/Resistor_SMD.3dshapes/R_0805_2012Metric.wrl"
+      (offset (xyz 0 0 0))
+      (scale (xyz 1 1 1))
+      (rotate (xyz 0 0 0))
+    )
+  )
   (footprint "Capacitor_SMD:C_0805_2012Metric_Pad1.18x1.45mm_HandSolder" (layer "F.Cu")
     (at 131.2 94.15 180)
@@
   (via (at 134.7 98.1) (size 0.85) (drill 0.25) (layers "F.Cu" "B.Cu") (net 1))
   (segment (start 135.2 100.2) (end 134.7 99.7) (width 0.4) (layer "In1.Cu") (net 1))
-  (segment (start 148.825 97.1) (end 141.4 97.1) (width 0.4) (layer "In1.Cu") (net 1))
   (segment (start 133.735 97.135) (end 134.7 98.1) (width 0.4) (layer "In1.Cu") (net 1))
+  (segment (start 139.3 100.2) (end 135.2 100.2) (width 0.4) (layer "In1.Cu") (net 1))
+  (segment (start 142.4 97.1) (end 139.3 100.2) (width 0.4) (layer "In1.Cu") (net 1))
+  (segment (start 148.825 97.1) (end 142.4 97.1) (width 0.4) (layer "In1.Cu") (net 1))
+  (segment (start 131.775 97.135) (end 133.735 97.135) (width 0.4) (layer "In1.Cu") (net 1))
   (segment (start 134.7 99.7) (end 134.7 98.1) (width 0.4) (layer "In1.Cu") (net 1))
-  (segment (start 141.4 97.1) (end 138.3 100.2) (width 0.4) (layer "In1.Cu") (net 1))
-  (segment (start 138.3 100.2) (end 135.2 100.2) (width 0.4) (layer "In1.Cu") (net 1))
-  (segment (start 131.775 97.135) (end 133.735 97.135) (width 0.4) (layer "In1.Cu") (net 1))
   (via (at 132.25 83.95) (size 0.85) (drill 0.25) (layers "F.Cu" "B.Cu") (free) (net 2))
   (via (at 125.1 97.95) (size 0.85) (drill 0.25) (layers "F.Cu" "B.Cu") (free) (net 2))
   (via (at 133.85 86.1) (size 0.85) (drill 0.25) (layers "F.Cu" "B.Cu") (free) (net 2))
+  (via (at 153.4 83.4) (size 0.85) (drill 0.25) (layers "F.Cu" "B.Cu") (free) (net 2))
   (via (at 144.35 88.25) (size 0.85) (drill 0.25) (layers "F.Cu" "B.Cu") (net 2))
   (via (at 155.5 89.75) (size 0.85) (drill 0.25) (layers "F.Cu" "B.Cu") (net 2))
@@
   (via (at 149.5 90.7) (size 0.85) (drill 0.25) (layers "F.Cu" "B.Cu") (free) (net 2))
   (via (at 130.15 94.2) (size 0.85) (drill 0.25) (layers "F.Cu" "B.Cu") (net 2))
+  (via (at 129.2 96.5) (size 0.85) (drill 0.25) (layers "F.Cu" "B.Cu") (free) (net 2))
   (via (at 152.8 90.1) (size 0.85) (drill 0.25) (layers "F.Cu" "B.Cu") (free) (net 2))
+  (via (at 136.2 96.5) (size 0.85) (drill 0.25) (layers "F.Cu" "B.Cu") (free) (net 2))
   (via (at 146.3 96.2) (size 0.85) (drill 0.25) (layers "F.Cu" "B.Cu") (free) (net 2))
   (via (at 137.8 84.6) (size 0.85) (drill 0.25) (layers "F.Cu" "B.Cu") (free) (net 2))
   (via (at 130.45 88.5) (size 0.85) (drill 0.25) (layers "F.Cu" "B.Cu") (net 2))
   (via (at 127 86.95) (size 0.85) (drill 0.25) (layers "F.Cu" "B.Cu") (free) (net 2))
+  (via (at 146.9 87) (size 0.85) (drill 0.25) (layers "F.Cu" "B.Cu") (free) (net 2))
+  (via (at 155.6 99.8) (size 0.85) (drill 0.25) (layers "F.Cu" "B.Cu") (free) (net 2))
   (segment (start 137.0375 98.85) (end 138.7125 98.85) (width 0.3) (layer "F.Cu") (net 3))
   (segment (start 138.7125 98.85) (end 139 98.5625) (width 0.3) (layer "F.Cu") (net 3))
   (via (at 149.5 87.05) (size 0.85) (drill 0.25) (layers "F.Cu" "B.Cu") (net 3))
   (via (at 149.5 89.2) (size 0.85) (drill 0.25) (layers "F.Cu" "B.Cu") (net 3))
-  (via (at 138.55 98.25) (size 0.85) (drill 0.25) (layers "F.Cu" "B.Cu") (net 3))
+  (via (at 138.5 98.2) (size 0.85) (drill 0.25) (layers "F.Cu" "B.Cu") (net 3))
   (segment (start 141.95 98.25) (end 147.2 93) (width 0.3) (layer "In2.Cu") (net 3))
   (segment (start 148 89.3) (end 149.4 89.3) (width 0.3) (layer "In2.Cu") (net 3))
@@
   (segment (start 146.7 93.5) (end 146.1 92.9) (width 0.2) (layer "F.Cu") (net 12))
   (segment (start 146.1 92.3) (end 145.85 92.05) (width 0.2) (layer "F.Cu") (net 12))
-  (segment (start 139.76 95.86) (end 142.7 98.8) (width 0.2) (layer "F.Cu") (net 13))
-  (segment (start 142.7 98.8) (end 143.5625 98.8) (width 0.2) (layer "F.Cu") (net 13))
   (segment (start 139.425 95.86) (end 139.76 95.86) (width 0.2) (layer "F.Cu") (net 13))
+  (segment (start 139.76 95.86) (end 141.5 97.6) (width 0.2) (layer "F.Cu") (net 13))
+  (segment (start 141.7 98.8) (end 141.5 98.6) (width 0.2) (layer "F.Cu") (net 13))
+  (segment (start 141.5 97.6) (end 141.5 98.6) (width 0.2) (layer "F.Cu") (net 13))
+  (segment (start 143.5625 98.8) (end 141.7 98.8) (width 0.2) (layer "F.Cu") (net 13))
   (segment (start 137.2 93.9) (end 136.95 94.15) (width 0.2) (layer "F.Cu") (net 14))
   (segment (start 137.2 91.4) (end 137.2 93.9) (width 0.2) (layer "F.Cu") (net 14))

Commit message: PCB: swap the MCU to 16F18326
Parts:
- U2: value PIC16F1825 -> PIC16F18326
Changed lines of the file:
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@@
       (effects (font (size 1 1) (thickness 0.15)))
     )
-    (fp_text value "PIC16F1825" (at 0 5.28) (layer "F.Fab")
+    (fp_text value "PIC16F18326" (at 0 5.28) (layer "F.Fab")
       (effects (font (size 1 1) (thickness 0.15)))
     )
